Commit message: new commit

File: src/articubot_one/description/robot_core.xacro (robot description, xacro)
@@ -15,4 +15,7 @@
   <material name="black">
     <color rgba="0 0 0 1"/>
+  </material>
+  <material name="red">
+    <color rgba="1 0 0 1"/>
   </material>
   <!-- It is preferred to define materials in a different file -->
