Commit message: new change

File: src/articubot_one/description/lidar.xacro (robot description, xacro)
@@ -1,8 +1,9 @@
 <?xml version="1.0"?>
 <robot xmlns:xacro="http://www.ros.org/wiki/xacro" name="robot">
+  <!-- creating the sensor body  -->
    <joint name ="laser_joint" type="fixed">
      <parent link="chassis"/>
      <child link="laser_frame"/>
-     <orgin xyz="0.1 0 0.175" rpy="0 0 0"/>
+     <origin xyz="0.1 0 0.175" rpy="0 0 0"/>
    </joint>
   <link name="laser_frame">
@@ -17,5 +18,4 @@
         <cylinder radius="0.05" length="0.04"/>
       </geometry>
-      <material name="blue"/>
     </collision>
     <xacro:inertial_cylinder mass="0.1" length="0.04" radius="0.05">
@@ -28,5 +28,5 @@
         <sensor name="laser" type="ray">
             <pose> 0 0 0 0 0 0 </pose>
-            <visualize>true</visualize>
+            <visualize>false</visualize>  <!--make it false if u dont want to see the laser scan patterns in gazebo-->
             <update_rate>10</update_rate>
             <ray>

File: src/articubot_one/description/robot.urdf.xacro (robot description, xacro)
@@ -2,3 +2,6 @@
 <robot xmlns:xacro="http://www.ros.org/wiki/xacro" name="robot">
    <xacro:include filename="robot_core.xacro"/>
+   <xacro:include filename="gazebo_control.xacro"/>
+   <xacro:include filename="lidar.xacro"/>
+   <xacro:include filename="camera.xacro"/>
 </robot>

File: src/articubot_one/description/robot_core.xacro (robot description, xacro)
@@ -49,4 +49,32 @@
     </xacro:inertial_box>
   </link>
+<!-- caster wheel -->
+  <joint name="caster_wheel_joint" type="fixed">
+    <parent link="chassis"/>
+    <child link="caster_wheel"/>
+    <origin xyz="0.24 0 0"/>
+  </joint>
+  <link name="caster_wheel">
+    <visual>
+      <geometry>
+       <sphere radius="0.05"/>
+      </geometry>
+      <material name="black"/>
+    </visual>
+    <collision>
+      <geometry>
+       <sphere radius="0.05"/>
+      </geometry>
+      <material name="black"/>
+    </collision>
+    <xacro:inertial_sphere mass="0.1" radius="0.05">
+      <origin xyz="0 0 0" rpy="0 0 0"/>
+    </xacro:inertial_sphere>
+  </link>
+  <gazebo reference="caster_wheel">
+    <material>Gazebo/Black</material>
+    <mu1 value="0.001"/>
+    <mu2 value="0.001"/>
+</gazebo>
   <!-- Left wheel link -->
   <joint name="left_wheel_joint" type="continuous">
@@ -67,5 +95,5 @@
         <cylinder radius="0.05" length="0.04"/>
       </geometry>
-      <material name="blue"/>
+      <material name="green"/>
     </collision>
     <xacro:inertial_cylinder mass="0.1" length="0.04" radius="0.05">
@@ -73,15 +101,12 @@
     </xacro:inertial_cylinder>
   </link>
-  <gazeebo reference ="left_wheel">
-    <material>Gazeebo/blue</material>
-  </gazeebo>
   <!-- Right wheel link -->
-  <joint name="Right_wheel_joint" type="continuous">
+  <joint name="right_wheel_joint" type="continuous">
     <parent link="base_link"/>
-    <child link="Right_wheel"/>
+    <child link="right_wheel"/>
     <origin xyz="0 -0.175 0" rpy="${pi/2} 0 0"/> <!-- By default, a cylinder is formed such that the flat surface is facing the z-axis, so we have to rotate it so that its z-axis coincides with the y-axis of the base_link -->
     <axis xyz="0 0 1"/> <!-- Rotate around z-axis -->
   </joint>
-  <link name="Right_wheel">
+  <link name="right_wheel">
     <visual>
       <geometry>
@@ -94,5 +119,5 @@
         <cylinder radius="0.05" length="0.04"/>
       </geometry>
-      <material name="blue"/>
+      <material name="green"/>
     </collision>
     <xacro:inertial_cylinder mass="0.1" length="0.04" radius="0.05">
@@ -100,32 +125,9 @@
     </xacro:inertial_cylinder>
   </link>
-  <gazeebo reference ="right_wheel">
-    <material>Gazeebo/blue</material>
-  </gazeebo>
-  <!-- caster wheel -->
-  <joint name="caster_wheel_joint" type="fixed">
-    <parent link="chassis"/>
-    <child link="caster_wheel"/>
-    <origin xyz="0.24 0 0"/>
-  </joint>
-  <link name="caster_wheel">
-    <visual>
-      <geometry>
-       <sphere radius="0.05"/>
-      </geometry>
-      <material name="black"/>
-    </visual>
-    <collision>
-      <geometry>
-       <sphere radius="0.05"/>
-      </geometry>
-      <material name="black"/>
-    </collision>
-    <xacro:inertial_sphere mass ="0.1" radius="0.05">
-      <origin xyz="0 0 0" rpy="0 0 0"/>
-    </xacro:inertial_sphere>
-  </link>
-  <gazeebo reference ="caster_wheel">
-    <material>Gazeebo/black</material>
-   </gazeebo>
+  <gazebo reference="right_wheel">
+    <material>Gazebo/Green</material>
+  </gazebo>
+  <gazebo reference="left_wheel">
+    <material>Gazebo/Green</material>
+  </gazebo>
 </robot>
